File: src/pcb/transmitter-pcb/transmitter-pcb.kicad_sch (KiCad schematic)
At the start: 5 parts

Commit message: adding new info
Parts:
- C1: renamed from C?; footprint (none) -> Capacitor_SMD:CP_Elec_3x5.3
- J1: renamed from J?; footprint (none) -> Connector_Wire:SolderWire-0.1sqmm_1x02_P3.6mm_D0.4mm_OD1mm
- U2: renamed from U?; footprint MODULE -> RF_Module:nRF24L01_Breakout
- gave numbers to parts that had none: 2
Connections:
- net at C1.2, J1.2 (Pin_2), U1.2 (GND)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: no longer A1.29 (GND), A1.4 (GND)
- new net: A1.29 (GND), A1.4 (GND)
Changed lines of the file:
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@@
   (junction (at 86.36 44.45) (diameter 0) (color 0 0 0 0)
   )
-  (junction (at 59.69 74.93) (diameter 0) (color 0 0 0 0)
-  )
   (wire (pts (xy 148.59 55.88) (xy 148.59 27.94))
     (stroke (width 0) (type default) (color 0 0 0 0))
@@
     (stroke (width 0) (type default) (color 0 0 0 0))
   )
-  (wire (pts (xy 59.69 74.93) (xy 59.69 99.06))
+  (wire (pts (xy 59.69 48.26) (xy 59.69 99.06))
     (stroke (width 0) (type default) (color 0 0 0 0))
   )
@@
     (stroke (width 0) (type default) (color 0 0 0 0))
   )
-  (wire (pts (xy 59.69 48.26) (xy 59.69 74.93))
-    (stroke (width 0) (type default) (color 0 0 0 0))
-  )
   (wire (pts (xy 104.14 39.37) (xy 104.14 53.34))
     (stroke (width 0) (type default) (color 0 0 0 0))
@@
     (stroke (width 0) (type default) (color 0 0 0 0))
   )
-  (wire (pts (xy 59.69 74.93) (xy 62.23 74.93))
-    (stroke (width 0) (type default) (color 0 0 0 0))
-  )
   (wire (pts (xy 86.36 48.26) (xy 67.31 48.26))
     (stroke (width 0) (type default) (color 0 0 0 0))
@@
   (symbol (lib_id "nRF24L01+:nRF24L01+") (at 123.19 33.02 0) (unit 1)
     (in_bom yes) (on_board yes) (fields_autoplaced)
-    (property "Reference" "U?" (id 0) (at 123.19 19.05 0))
+    (property "Reference" "U2" (id 0) (at 123.19 19.05 0))
     (property "Value" "nRF24L01+" (id 1) (at 123.19 21.59 0))
-    (property "Footprint" "MODULE" (id 2) (at 123.19 30.48 0)
+    (property "Footprint" "RF_Module:nRF24L01_Breakout" (id 2) (at 123.19 30.48 0)
       (effects (font (size 1.27 1.27)) hide)
     )
@@
   (symbol (lib_id "MCU_Module:Arduino_Nano_Every") (at 87.63 74.93 270) (unit 1)
     (in_bom yes) (on_board yes)
-    (property "Reference" "A?" (id 0) (at 53.34 78.5114 90))
+    (property "Reference" "A1" (id 0) (at 53.34 78.5114 90))
     (property "Value" "Arduino_Nano_Every" (id 1) (at 53.34 75.9714 90))
     (property "Footprint" "Module:Arduino_Nano" (id 2) (at 87.63 74.93 0)
@@
   (symbol (lib_id "Regulator_Linear:L78L33_SO8") (at 86.36 27.94 0) (unit 1)
     (in_bom yes) (on_board yes) (fields_autoplaced)
-    (property "Reference" "U?" (id 0) (at 86.36 20.32 0))
+    (property "Reference" "U1" (id 0) (at 86.36 20.32 0))
     (property "Value" "L78L33_SO8" (id 1) (at 86.36 22.86 0))
     (property "Footprint" "Package_SO:SOIC-8_3.9x4.9mm_P1.27mm" (id 2) (at 88.9 22.86 0)
@@
   (symbol (lib_id "Device:C_Polarized_US") (at 67.31 39.37 0) (unit 1)
     (in_bom yes) (on_board yes) (fields_autoplaced)
-    (property "Reference" "C?" (id 0) (at 71.12 37.4649 0)
+    (property "Reference" "C1" (id 0) (at 71.12 37.4649 0)
       (effects (font (size 1.27 1.27)) (justify left))
     )
@@
       (effects (font (size 1.27 1.27)) (justify left))
     )
-    (property "Footprint" "" (id 2) (at 67.31 39.37 0)
+    (property "Footprint" "Capacitor_SMD:CP_Elec_3x5.3" (id 2) (at 67.31 39.37 0)
       (effects (font (size 1.27 1.27)) hide)
     )
@@
   (symbol (lib_id "Connector:Conn_01x02_Male") (at 92.71 110.49 90) (unit 1)
     (in_bom yes) (on_board yes) (fields_autoplaced)
-    (property "Reference" "J?" (id 0) (at 96.52 108.5849 90)
+    (property "Reference" "J1" (id 0) (at 96.52 108.5849 90)
       (effects (font (size 1.27 1.27)) (justify right))
     )
@@
       (effects (font (size 1.27 1.27)) (justify right))
     )
-    (property "Footprint" "" (id 2) (at 92.71 110.49 0)
+    (property "Footprint" "Connector_Wire:SolderWire-0.1sqmm_1x02_P3.6mm_D0.4mm_OD1mm" (id 2) (at 92.71 110.49 0)
       (effects (font (size 1.27 1.27)) hide)
     )
@@
   (symbol_instances
     (path "/1ecb9880-bf55-4540-a79f-60dbfc5b425f"
-      (reference "A?") (unit 1) (value "Arduino_Nano_Every") (footprint "Module:Arduino_Nano")
+      (reference "A1") (unit 1) (value "Arduino_Nano_Every") (footprint "Module:Arduino_Nano")
     )
     (path "/56d4433a-1559-4d3a-923e-e55aa8259441"
-      (reference "C?") (unit 1) (value "C_Polarized_US") (footprint "")
+      (reference "C1") (unit 1) (value "C_Polarized_US") (footprint "Capacitor_SMD:CP_Elec_3x5.3")
     )
     (path "/f1969937-85de-4110-98d5-b8997e427f55"
-      (reference "J?") (unit 1) (value "Conn_01x02_Male") (footprint "Connector_Coaxial:SMA_Amphenol_132203-12_Horizontal")
+      (reference "J1") (unit 1) (value "Conn_01x02_Male") (footprint "Connector_Wire:SolderWire-0.1sqmm_1x02_P3.6mm_D0.4mm_OD1mm")
+    )
+    (path "/3af2520d-df70-423f-ac99-ef6619de0a0c"
+      (reference "U1") (unit 1) (value "L78L33_SO8") (footprint "Package_SO:SOIC-8_3.9x4.9mm_P1.27mm")
     )
     (path "/14af66e1-eae3-4c4d-bfee-92f0d3466a73"
-      (reference "U?") (unit 1) (value "nRF24L01+") (footprint "MODULE")
-    )
-    (path "/3af2520d-df70-423f-ac99-ef6619de0a0c"
-      (reference "U?") (unit 1) (value "L78L33_SO8") (footprint "Package_SO:SOIC-8_3.9x4.9mm_P1.27mm")
-    )
-  )
+      (reference "U2") (unit 1) (value "nRF24L01+") (footprint "RF_Module:nRF24L01_Breakout")
+    )
+  )
